File: frodo_power_module.kicad_pcb (KiCad board)
At the start: 2 copper layers, 88 x 69 mm, 84 parts, among them J1 Keystone 1048, J10 SWD Header, J2 Molex MicroFit 2x3, J3 Molex MicroFit 2x2, J4 Molex MicroFit 2x2, J5 JST-GH, J6 JST-GH, J7 Molex MicroFit 2x3, U1 STM32F042F6Px, U2 L7805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

Commit message: Add finishing touches, generate fabrication files
Parts:
- added G***: LOGO, frodo_power_module:rapid_logo, B.Cu at (126.9, 109.4)
- C23, C24, C25: moved to B.Cu
- Y1: footprint Oscillator:Oscillator_SMD_SeikoEpson_SG210-4Pin_2.5x2.0mm -> Crystal:Crystal_SMD_5032-4Pin_5.0x3.2mm
- moved TH1 41.5 mm to (58.5, 105.0)
- moved C24 34.8 mm to (85.1, 128.0), turned to 90 degrees
- moved R26 28.0 mm to (71.5, 72.4), turned to -90 degrees
- moved R25 25.9 mm to (69.6, 72.4), turned to -90 degrees
- moved D3 25.7 mm to (71.5, 75.7), turned to 90 degrees
- moved D2 24.0 mm to (69.6, 75.7), turned to 90 degrees
- moved J10 11.7 mm to (131.5, 129.6), turned to 180 degrees
- moved C25 8.56 mm to (116.8, 124.7)
- moved R21 5.30 mm to (117.5, 130.2), turned to 180 degrees
- moved R23 5.01 mm to (117.2, 119.7), turned to 180 degrees
- moved C23 2.18 mm to (76.9, 121.9), turned to -90 degrees
- moved R24 2.10 mm to (82.0, 106.7)
- moved R6 2.06 mm to (82.0, 103.5)
- moved R20 0.88 mm to (117.5, 128.5)
Routing:
- net Net-(D3-K): track 14.8 -> 59.0 mm
- net Net-(D1-K): track 47.7 -> 88.4 mm
- net Net-(D2-K): track 25.5 -> 63.0 mm
- net +VSW: track 41.6 -> 27.4 mm
- net +3V3: track 99.2 -> 112.5 mm
- net SWDIO: track 42.5 -> 50.3 mm
- net GND: track 69.3 -> 76.9 mm, vias 31 -> 36
- net Net-(R10-Pad2): track 32.6 -> 39.5 mm
- net SWCLK: track 44.1 -> 49.1 mm
- net VSENSE_BATT: track 35.1 -> 33.2 mm
- net VDC: track 56.0 -> 57.7 mm
- net Net-(U4-VSET): track 3.98 -> 2.39 mm
- net VSENSE_CHARGE: track 41.9 -> 41.2 mm
Other:
- board text added: "FRoDO Power Module"
- board text added: "JLCJLCJLCJLC"
- board text added: "rev 2"
