File: control_logic.kicad_sch (KiCad schematic)
At the start: 71 parts, among them J8 TC2050, J9 SWD Header, U1 AZ1117I-3.3, U2 TPD4E1U06, U3 MCP2562-E-SN, U4 L7805, U5 STM32F105RCTx, Y1 8MHz 12pF

Commit message: cleanup and export 3d-models
Parts:
- removed C10, C18, C19, C20, C21, C22: 100n, Capacitor_SMD:C_0402_1005Metric, symbol Device:C
- removed C11: 10u, Capacitor_SMD:C_1206_3216Metric, symbol Device:C_Small
- removed C12: 22u, Capacitor_SMD:C_1206_3216Metric, symbol Device:C_Small
- removed C13: 330n, Capacitor_SMD:C_0603_1608Metric, symbol Device:C_Small
- removed C14, C15, C16: 100n, Capacitor_SMD:C_0402_1005Metric, symbol Device:C_Small
- removed C17: 4u7, Capacitor_SMD:C_0402_1005Metric, symbol Device:C
- removed C23, C27: 10n, Capacitor_SMD:C_0402_1005Metric, symbol Device:C
- removed C24, C26: 1u, Capacitor_SMD:C_0402_1005Metric, symbol Device:C
- removed C25, C28: 10p, Capacitor_SMD:C_0402_1005Metric, symbol Device:C
- removed D10, D11, D12, D8, D9: green, LED_SMD:LED_0805_2012Metric, symbol Device:LED_Small
- removed D4, D5: (no value), Diode_SMD:D_SMA, symbol Device:D_Schottky
- removed D6: red, LED_SMD:LED_0603_1608Metric, symbol Device:LED_Small
- removed D7: yellow, LED_SMD:LED_0805_2012Metric, symbol Device:LED_Small
- removed FB1: 120R, Inductor_SMD:L_0603_1608Metric, symbol Device:FerriteBead
- removed J8: TC2050, Connector:Tag-Connect_TC2050-IDC-FP_2x05_P1.27mm_Vertical, symbol Connector_Generic:Conn_02x05_Counter_Clockwise
- removed J9: SWD Header, Connector_PinHeader_2.54mm:PinHeader_1x04_P2.54mm_Vertical_SMD_Pin1Left, symbol Connector_Generic:Conn_01x04
- removed R1, R2, R3, R6, R7, R9: 22R, Resistor_SMD:R_0402_1005Metric, symbol Device:R_Small
- removed R10: 68k, Resistor_SMD:R_0603_1608Metric, symbol Device:R
- removed R11, R13, R4, R5: 10k, Resistor_SMD:R_0402_1005Metric, symbol Device:R
- removed R12: 30k, Resistor_SMD:R_0603_1608Metric, symbol Device:R
- removed R14, R16, R17, R18, R19, R20, R21, R22: 1k, Resistor_SMD:R_0402_1005Metric, symbol Device:R_Small
- removed R15: 100k, Resistor_SMD:R_0402_1005Metric, symbol Device:R_Small
- removed R23: 1k, Resistor_SMD:R_0402_1005Metric, symbol Device:R
- removed R8: 120, Capacitor_SMD:C_0402_1005Metric, symbol Device:R_Small
- removed SW1, SW2: (no value), Button_Switch_SMD:SW_SPST_TS-1088-xR020, symbol Switch:SW_SPST
- removed TP10, TP11, TP12, TP13, TP5, TP6, TP7, TP8, TP9: TestPoint, TestPoint:TestPoint_Pad_D2.0mm, symbol Connector:TestPoint
- removed U1: AZ1117I-3.3, Package_TO_SOT_SMD:SOT-223-3_TabPin2, symbol Regulator_Linear:AZ1117-3.3
- removed U2: TPD4E1U06, Package_TO_SOT_SMD:SOT-563, symbol stigma:TPD4E001DRL
- removed U3: MCP2562-E-SN, Package_SO:SOIC-8_3.9x4.9mm_P1.27mm, symbol Interface_CAN_LIN:MCP2562-E-SN
- removed U4: L7805, Package_TO_SOT_SMD:TO-252-2, symbol Regulator_Linear:L7805
- removed U5: STM32F105RCTx, Package_QFP:LQFP-64_10x10mm_P0.5mm, symbol MCU_ST_STM32F1:STM32F105RCTx
- removed Y1: 8MHz 12pF, Crystal:Crystal_SMD_5032-4Pin_5.0x3.2mm, symbol Device:Crystal_GND24
Connections:
- no-connect marks 30 -> 0
Other:
- note removed: "12,6V"
- note removed: "24V"
- note removed: "ADC12_IN2"
- note removed: "ADC12_IN3"
- note removed: "ADC12_IN4"
- note removed: "CAN"
- note removed: "Charge Indicator LEDs"
- note removed: "Clock"
- note removed: "DNP"
- note removed: "INFO: those pins support CAN bootloader"
- note removed: "LEDs"
- note removed: "ONLY 3V3 capable"
- note removed: "Regulators"
- note removed: "Sensing"
- note removed: "V_CH_s/24V = R19/(R18+R19) V_CH_s_max = 3v3; R19 = 10k -> R18 ~ 68k"
- note removed: "V_SNS/12.6V = R21/(R20+R21) V_SNS_max = 3v3; R21 = 10k -> R20 = 30k"
- note removed: "controller"
- note removed: "from batteries"
- note removed: "programming adapters"
- note removed: "redundand but does not hurt"
